Commit message: Modified urdf, added color iin gazebo and added launch file for robot in  warehouse world

File: my_rb1_description/urdf/my_rb1_robot.urdf (robot description, URDF)
Before this commit: robot my_rb1_robot, 7 links, 6 joints
Links:
- link base_footprint: mass None -> 0.0001; geometry visual box size=0.001 0.001 0.001
- link left_wheel: geometry collision cylinder length=0.025 radius=0.025; visual cylinder length=0.025 radius=0.025
- link right_wheel: geometry collision cylinder length=0.025 radius=0.025; visual cylinder length=0.025 radius=0.025

Commit message: Added plugins for differential drive and laser sensor

File: my_rb1_description/urdf/my_rb1_robot.urdf (robot description, URDF)
Before this commit: robot my_rb1_robot, 7 links, 6 joints
Links:
- link front_laser: mass None -> 0.1
- link left_wheel: geometry collision cylinder length=0.05 radius=0.025; visual cylinder length=0.05 radius=0.025
- link right_wheel: geometry collision cylinder length=0.05 radius=0.025; visual cylinder length=0.05 radius=0.025

Commit message: modified diff drive plugin and wheel mass, inertia

File: my_rb1_description/urdf/my_rb1_robot.urdf (robot description, URDF)
Before this commit: robot my_rb1_robot, 7 links, 6 joints
Links:
- link left_wheel: mass 0.5 -> 1.0
- link right_wheel: mass 0.5 -> 1.0
